File: NXP/Hardware/NXP_SBC/Ethernet.kicad_sch (KiCad schematic)
At the start: 34 parts, among them J4 RJ45_Wuerth_7499010121A, U7 KSZ8081RNBIA-TR

Commit message: More additions to schematic
Connections:
- net +3V3: no longer C56.1, C57.2, C58.2, R10.1, R49.1, R50.1, R53.1, R55.1, R57.1, R59.1, R61.1, R7.1, R8.1, U7.17 (VDDIO)
- net ETH_CONFIG2 renamed ETH_CRS_DV
- new net DCDC_3V3: C56.1, C57.2, C58.2, R10.1, R49.1, R50.1, R53.1, R55.1, R57.1, R59.1, R61.1, R7.1, R8.1, U7.17 (VDDIO)
Other:
- note added: "EVAL HAS RST GOING TO SHIFT REG CAN I JUST USE GPIO?"

Commit message: minor updates
Connections:
- net +3V3 is gone; now on net DCDC_3V3: J4.10, J4.12, U7.3 (VDDA_3.3)
