File: NXP/Hardware/NXP_SBC/Memory_sch.kicad_sch (KiCad schematic)
At the start: 15 parts, among them J1 Micro_SD_Card_Det2, U2 MT41K256M16TW-107_P_TR

Commit message: Added some more to the DDR memory schematic
Upgraded the project to kicad 9.0
Parts:
- added C27, C28, C29, C30, C31, C32, C33, C34, C35, C36, C37, C38: 220nF, Capacitor_SMD:C_0603_1608Metric_Pad1.08x0.95mm_HandSolder, symbol Device:C_Small
- added C39, C40: 100nF, Capacitor_SMD:C_0603_1608Metric_Pad1.08x0.95mm_HandSolder, symbol Device:C_Small
- added C41: 4u7F, Capacitor_SMD:C_0603_1608Metric_Pad1.08x0.95mm_HandSolder, symbol Device:C_Small
- added C42, C43, C44, C45: 2p2F, Capacitor_SMD:C_0603_1608Metric_Pad1.08x0.95mm_HandSolder, symbol Device:C_Small
- added R41: 1k5, 1%, Resistor_SMD:R_0603_1608Metric, symbol Device:R_Small
- added R42: 1k, 1%, Resistor_SMD:R_0603_1608Metric, symbol Device:R_Small
- added R43: 240R, Resistor_SMD:R_0603_1608Metric, symbol Device:R_Small
- added R44: 470R, Resistor_SMD:R_0603_1608Metric, symbol Device:R_Small
Connections:
- net GND: now also U2.A9 (VSS_1), U2.B1 (VSSQ_1), U2.B3 (VSS_2), U2.B9 (VSSQ_2), U2.D1 (VSSQ_3), U2.D8 (VSSQ_4), U2.E1 (VSS_3), U2.E2 (VSSQ_5), U2.E8 (VSSQ_6), U2.F9 (VSSQ_7), U2.G1 (VSSQ_8), U2.G8 (VSS_4), U2.G9 (VSSQ_9), U2.J2 (VSS_5), U2.J8 (VSS_6), U2.M1 (VSS_7), U2.M9 (VSS_8), U2.P1 (VSS_9), U2.P9 (VSS_10), U2.T1 (VSS_11), U2.T9 (VSS_12), C27.2, C28.2, C29.2, C30.2, C31.2, C32.2, C33.2, C34.2, C35.2, C36.2, C37.2, C38.2, C40.2, C41.2, R42.2, R43.2
- net RAM_CK: now also R44.2
- net RAM_CK#: now also R44.1
- net RAM_DQ9: now also C42.1, C43.1
- net RAM_LDQS: now also C44.1, C45.1
- net RAM_LDQS#: now also C44.2, C45.2
- net RAM_UDQS#: now also C42.2, C43.2
- net +1V35: now reaches U2.A1 (VDDQ_1)
- net +1V35: now also U2.A8 (VDDQ_2), U2.B2 (VDD_1), U2.C1 (VDDQ_3), U2.C9 (VDDQ_4), U2.D2 (VDDQ_5), U2.D9 (VDD_2), U2.E9 (VDDQ_6), U2.F1 (VDDQ_7), U2.G7 (VDD_3), U2.H2 (VDDQ_8), U2.H9 (VDDQ_9), U2.K2 (VDD_4), U2.K8 (VDD_5), U2.N1 (VDD_6), U2.N9 (VDD_7), U2.R1 (VDD_8), U2.R9 (VDD_9), C27.1, C28.1, C29.1, C30.1, C31.1, C32.1, C33.1, C34.1, C35.1, C36.1, C37.1, C38.1, C39.1, C41.1, R41.1
- net DDR_VREF: now reaches U2.H1 (VREFDQ)
- net DDR_VREF: now also U2.M8 (VREFCA), C39.2, C40.1, R41.2, R42.1
- net RAM_ODT: now reaches U2.K1 (ODT)
- net RAM_ZQ: no longer names the net of U2.L8 (ZQ)
- net RAM_ZQ: now also R43.1
- no-connect marks 0 -> 5
Other:
- note added: "CLK TERMINATION CLOSE TO RAM CHIP"
- moved on the sheet: D1, D2, D3, D4, D5, D6, D7, J1, R1, R2, R3, R4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

Commit message: minor updates
Connections:
- net +3V3 renamed DCDC_3V3
Changed lines of the file:
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@@
+	)
+	(symbol
+		(lib_id "power:+1V35")
+		(at 412.75 80.01 0)
+		(unit 1)
+		(exclude_from_sim no)
+		(in_bom yes)
+		(on_board yes)
+		(dnp no)
+		(fields_autoplaced yes)
+		(property "Reference" "#PWR01"
+			(at 412.75 83.82 0)
+			(effects
+				(font
+					(size 1.27 1.27)
+				)
+				(hide yes)
+			)
+		)
+		(property "Value" "DCDC_3V3"
+			(at 412.75 74.93 0)
+			(effects
+				(font
+					(size 1.27 1.27)
+				)
+			)
+		)
+		(property "Footprint" ""
+			(at 412.75 80.01 0)
+			(effects
+				(font
+					(size 1.27 1.27)
+				)
+				(hide yes)
+			)
+		)
+		(property "Datasheet" ""
+			(at 412.75 80.01 0)
+			(effects
+				(font
+					(size 1.27 1.27)
+				)
+				(hide yes)
+			)
+		)
+		(property "Description" "Power symbol creates a global label with name \"+1V35\""
+			(at 412.75 80.01 0)
+			(effects
+				(font
+					(size 1.27 1.27)
+				)
+				(hide yes)
+			)
+		)
+		(pin "1"
+		)
+		(instances
+			(project "NXP_SBC"
+				(path "/e82fc437-413b-4185-b609-66f66e24e498/cf3598eb-c9d5-4140-bda5-3b7546e36109"
+					(reference "#PWR01")
+					(unit 1)
+				)
+			)
+		)
 	)
 	(symbol
@@
 					(unit 1)
 				)
-			)
-		)
-	)
-	(symbol
-		(lib_id "power:+3V3")
-		(at 412.75 80.01 0)
-		(unit 1)
-		(exclude_from_sim no)
-		(in_bom yes)
-		(on_board yes)
-		(dnp no)
-		(fields_autoplaced yes)
-		(property "Reference" "#PWR01"
-			(at 412.75 83.82 0)
-			(effects
-				(font
-					(size 1.27 1.27)
-				)
-				(hide yes)
-			)
-		)
-		(property "Value" "+3V3"
-			(at 412.75 74.93 0)
-			(effects
-				(font
-					(size 1.27 1.27)
-				)
-			)
-		)
-		(property "Footprint" ""
-			(at 412.75 80.01 0)
-			(effects
-				(font
-					(size 1.27 1.27)
-				)
-				(hide yes)
-			)
-		)
-		(property "Datasheet" ""
-			(at 412.75 80.01 0)
-			(effects
-				(font
-					(size 1.27 1.27)
-				)
-				(hide yes)
-			)
-		)
-		(property "Description" "Power symbol creates a global label with name \"+3V3\""
-			(at 412.75 80.01 0)
-			(effects
-				(font
-					(size 1.27 1.27)
-				)
-				(hide yes)
-			)
-		)
-		(pin "1"
-		)
-		(instances
-			(project "NXP_SBC"
-				(path "/e82fc437-413b-4185-b609-66f66e24e498/cf3598eb-c9d5-4140-bda5-3b7546e36109"
-					(reference "#PWR01")
-					(unit 1)
-				)
