File: NXP/Hardware/NXP_SBC/Audio.kicad_sch (KiCad schematic)
At the start: 17 parts, among them J10 Conn_01x02, J8 Conn_01x02, U10 WM8962BECSN_R

Commit message: Finished audio section
Parts:
- added C79, C84, C85, C86: 100nF, Capacitor_SMD:C_0603_1608Metric_Pad1.08x0.95mm_HandSolder, symbol Device:C_Small
- added C80, C81, C82, C83: 1nF, Capacitor_SMD:C_0603_1608Metric_Pad1.08x0.95mm_HandSolder, symbol Device:C_Small
- added C87, C88: 15pF, Capacitor_SMD:C_0603_1608Metric_Pad1.08x0.95mm_HandSolder, symbol Device:C_Small
- added C89, C92, C93, C94, C95: 1uF, Capacitor_SMD:C_0603_1608Metric_Pad1.08x0.95mm_HandSolder, symbol Device:C_Small
- added C90, C98, C99: 4u7F, Capacitor_SMD:C_0603_1608Metric_Pad1.08x0.95mm_HandSolder, symbol Device:C_Small
- added C91, C96, C97: 2u2F, Capacitor_SMD:C_0603_1608Metric_Pad1.08x0.95mm_HandSolder, symbol Device:C_Small
- added D10, D11, D12, D13: PESD3V3Z1BSFYL, symbol Chase_Diode:PESD3V3Z1BSFYL
- added J13, J14: Conn_01x03, symbol Connector_Generic:Conn_01x03
- added J9: AudioJack4_SwitchT1, Connector_Audio:Jack_3.5mm_CUI_SJ1-3535NG_Horizontal_CircularHoles, symbol Connector_Audio:AudioJack4_SwitchT1
- added R100, R97, R98: 1K, Resistor_SMD:R_01005_0402Metric, symbol Device:R_Small
- added R101, R102, R103, R104, R113, R114, R91, R92: 10K, Resistor_SMD:R_01005_0402Metric, symbol Device:R_Small
- added R105, R106, R107, R108, R109: 33R, Resistor_SMD:R_01005_0402Metric, symbol Device:R_Small
- added R110, R111, R112, R89, R90, R95, R96: 0R, Resistor_SMD:R_01005_0402Metric, symbol Device:R_Small
- added R93, R94: 20R, Resistor_SMD:R_01005_0402Metric, symbol Device:R_Small
- added R99: 1K2, Resistor_SMD:R_01005_0402Metric, symbol Device:R_Small
- added TP2, TP3: TestPoint, TestPoint:TestPoint_Pad_3.0x3.0mm, symbol Connector:TestPoint
Connections:
- net CIFMODE is gone; now on net GND: U10.F2 (CIFMODE)
- net DCDC_3V3: now also R113.2
- net GND: now also C79.2, C80.2, C81.2, C84.2, C87.2, C88.2, C89.2, C90.2, C96.2, C97.2, C98.2, D10.1 (K1), D11.1 (K1), D12.1 (K1), D13.1 (K1), J13.3 (Pin_3), J14.3 (Pin_3), J9.S, R101.1, R102.1, R103.1, R104.1, R114.1, R91.1, R92.1, R93.1, R94.1, R95.2, R96.2
- net GPIO5: now also R112.2, R114.2
- net HPOUTFB: now also R95.1
- net HPOUTL: now also C83.1, R89.1, R92.2
- net HPOUTR: now also C82.1, R90.1, R91.2
- net IN1L: now also C84.1, C85.1
- net IN1R: now also C79.1, C86.1
- net IN2L: now also C93.1, R101.2
- net IN2R: now also C92.1, R102.2
- net IN3L: now also C94.1, R103.2
- net IN3R: now also C95.1, R104.2
- net MICBIAS: now also C99.1, R98.2
- net SPKOUTLN: now also R82.1
- net SPKOUTLP: now also R81.1
- net SPKOUTRN: now also R86.1
- net SPKOUTRP: now also R85.1
- net ADCDAT: no longer names the net of U10.D2 (ADCDAT)
- net ADCDAT: now also R106.1
- net BCLK: no longer names the net of U10.E1 (BCLK)
- net BCLK: now also R108.2
- net CLKOUT3/GPIO3: no longer names the net of U10.F4 (CLKOUT3/GPIO3)
- net CLKOUT5: no longer names the net of U10.G6 (CLKOUT5)
- net CLKOUT5: now also TP3.1
- net CPCA: no longer names the net of U10.B6 (CPCA)
- net CPCA: now also C91.1
- net CPCB: no longer names the net of U10.B7 (CPCB)
- net CPCB: now also C91.2
- net CPVOUTN: no longer names the net of U10.A7 (CPVOUTN)
- net CPVOUTN: now also C96.1
- net CPVOUTP: no longer names the net of U10.A6 (CPVOUTP)
- net CPVOUTP: now also C97.1
- net DACDAT: no longer names the net of U10.D1 (DACDAT)
- net DACDAT: now also R105.1
- net IN4L: no longer names the net of U10.E6 (IN4L)
- net IN4R: no longer names the net of U10.E7 (IN4R)
- net LRCLK: no longer names the net of U10.D3 (LRCLK)
- net LRCLK: now also R107.1
- net MCLK/XTI: no longer names the net of U10.G7 (MCLK/XTI)
- net MCLK/XTI: now also R109.2
- net SCLK renamed CODEC_SCLK
- net SDA renamed CODEC_SDA
- net VMIDC: no longer names the net of U10.C5 (VMIDC)
- net VMIDC: now also C98.1
- net XTO: no longer names the net of U10.F7 (XTO)
- net XTO: now also TP2.1
- net ~{CS}/GPIO6: no longer names the net of U10.E3 (~{CS}/GPIO6)
- net ~{CS}/GPIO6: now also R110.2
- new net: C80.1, D11.2 (K2), J9.R1, R90.2
- new net: C81.1, D12.2 (K2), J9.T, R89.2
- new net: C82.2, R93.2
- new net: C89.1, C90.1, C99.2, R98.1, R99.2
- new net: C86.2, C87.1, C88.1, R100.2, R97.2, R99.1
- new net: C93.2, J13.1 (Pin_1)
- new net: C92.2, J13.2 (Pin_2)
- new net: C83.2, R94.2
- new net: C85.2, R96.1, R97.1
- new net: C94.2, J14.1 (Pin_1)
- new net: C95.2, J14.2 (Pin_2)
- new net CODEC_ADCDAT: R106.2
- new net CODEC_BCLK: R108.1
- new net CODEC_DACDAT: R105.2
- new net CODEC_INT: R110.1, R111.2
- new net CODEC_LRCLK: R107.2
- new net CODEC_MCLK: R109.1
- new net HP_DET: D13.2 (K2), J9.TN, R111.1, R112.1, R113.1
- new net HP_MIC: D10.2 (K2), J9.R2, R100.1
Other:
- note added: "CODEC"
- note added: "HEADSET"
- note added: "MIC BIAS"
- note added: "MISC INPUTS"
- note added: "SKR1"
- note added: "SKR2"
- note added: "SPEAKERS"
- moved on the sheet: C73, C74, C75, C76, C77, C78, J10, J8, R81, R82, R83, R84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

Commit message: Minor updates again!
Other:
- note added: "MICVDD SHOULD BE 2V5???"
Changed lines of the file:
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@@
 	(text "MAKE LOW NOISE SUPPLY"
 		(exclude_from_sim no)
-		(at 231.902 41.148 0)
+		(at 208.534 43.688 0)
 		(effects
 			(font
@@
 				(color 255 0 0 1)
 			)
+		)
+	)
+	(text "MICVDD SHOULD BE 2V5???\n"
+		(exclude_from_sim no)
+		(at 209.55 46.99 0)
+		(effects
+			(font
+				(size 1.27 1.27)
+				(color 255 0 0 1)
+			)
