File: NXP/Hardware/NXP_SBC/Power.kicad_sch (KiCad schematic)
At the start: 101 parts, among them J6 USB_C_Receptacle_PowerOnly_6P, J7 Screw_Terminal_01x02, Q1 DMN3150L-7, Q2 DMN3150L-7, Q3 DMN3150L-7, Q4 DMN3150L-7, Q5 DMN3150L-7, Q6 DMN3150L-7, Q8 DMN3150L-7, U11 AP3401, U3 AP3401, U4 AP3401, U5 MP2144GJ-P, U6 MAX811REUS-T, U9 AP3401

Commit message: Minor updates again!
Other:
- note added: "2A"
- note added: "MAKE 5V SUPPLY FOR SPEAKERS"
- note added: "MAKE LOW NOISE SUPPLY FOR CODEC"
- note added: "WHAT IS VDD_SNVS_3V3?"
Changed lines of the file:
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@@
 	(generator_version "9.0")
 	(paper "A2")
+	(text "2A"
+		(exclude_from_sim no)
+		(at 435.356 40.132 0)
+		(effects
+			(font
+				(size 1.27 1.27)
+				(thickness 0.254)
+				(bold yes)
+				(color 255 0 0 1)
+			)
+		)
+	)
+	(text "2A"
+		(exclude_from_sim no)
+		(at 430.276 203.454 0)
+		(effects
+			(font
+				(size 1.27 1.27)
+				(thickness 0.254)
+				(bold yes)
+				(color 255 0 0 1)
+			)
+		)
+	)
 	(text "PMIC_STBY_REQ = 0, GPIO_DVFS = 0, output is 1.4V (1.375V + 25mV)\nPMIC_STBY_REQ = 0, GPIO_DVFS = 1, output is 1.3V (1.275V + 25mV)\nPMIC_STBY_REQ = 1, GPIO_DVFS = 0, output is 0.925V (0.9V + 25mV)"
 		(exclude_from_sim no)
@@
 			)
 		)
+	)
+	(text "WHAT IS VDD_SNVS_3V3?"
+		(exclude_from_sim no)
+		(at 515.874 301.244 0)
+		(effects
+			(font
+				(size 2.54 2.54)
+				(thickness 0.254)
+				(bold yes)
+				(color 255 0 0 1)
+			)
+		)
+	)
+	(text "MAKE 5V SUPPLY FOR SPEAKERS"
+		(exclude_from_sim no)
+		(at 217.17 335.28 0)
+		(effects
+			(font
+				(size 1.27 1.27)
+				(color 255 0 0 1)
+			)
+		)
+	)
+	(text "2A"
+		(exclude_from_sim no)
+		(at 134.874 38.862 0)
+		(effects
+			(font
+				(size 1.27 1.27)
+				(thickness 0.254)
+				(bold yes)
+				(color 255 0 0 1)
+			)
+		)
+	)
+	(text "2A"
+		(exclude_from_sim no)
+		(at 432.562 119.634 0)
+		(effects
+			(font
+				(size 1.27 1.27)
+				(thickness 0.254)
+				(bold yes)
+				(color 255 0 0 1)
+			)
+		)
+	)
+	(text "2A"
+		(exclude_from_sim no)
+		(at 143.256 166.37 0)
+		(effects
+			(font
+				(size 1.27 1.27)
+				(thickness 0.254)
+				(bold yes)
+				(color 255 0 0 1)
+			)
+		)
+	)
+	(text "MAKE LOW NOISE SUPPLY FOR CODEC"
+		(exclude_from_sim no)
+		(at 219.456 337.566 0)
+		(effects
+			(font
+				(size 1.27 1.27)
+				(color 255 0 0 1)
+			)
+		)
