File: NXP/Hardware/NXP_SBC/Processor.kicad_sch (KiCad schematic)
At the start: 33 parts, among them U1 MCIMX6Y2DVM09AB

Commit message: minor updates
Connections:
- net uP_GPIO4_IO12: now reaches U1.A3 (NAND_READY_B)
- net uP_GPIO4_IO15: now reaches U1.A4 (NAND_CLE)
- net uP_GPIO4_IO10: now reaches U1.B4 (NAND_ALE)
- net uP_GPIO4_IO11: now reaches U1.D5 (NAND_WP_B)
- net RADIO_SD_CLK renamed uP_SD2_CLK
- net RADIO_SD_CMD renamed uP_SD2_CMD
- net RADIO_SD_DATA0 renamed uP_SD2_DATA0
- net RADIO_SD_DATA1 renamed uP_SD2_DATA1
- net RADIO_SD_DATA2 renamed uP_SD2_DATA2
- net RADIO_SD_DATA3 renamed uP_SD2_DATA3
Changed lines of the file:
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@@
 	(wire
 		(pts
+			(xy 154.94 490.22) (xy 177.8 490.22)
+		)
+		(stroke
+			(width 0)
+			(type default)
+		)
+	)
+	(wire
+		(pts
 			(xy 549.91 146.05) (xy 567.69 146.05)
 		)
@@
 	(wire
 		(pts
+			(xy 154.94 502.92) (xy 177.8 502.92)
+		)
+		(stroke
+			(width 0)
+			(type default)
+		)
+	)
+	(wire
+		(pts
 			(xy 680.72 156.21) (xy 641.35 156.21)
 		)
@@
 	(wire
 		(pts
+			(xy 154.94 500.38) (xy 177.8 500.38)
+		)
+		(stroke
+			(width 0)
+			(type default)
+		)
+	)
+	(wire
+		(pts
 			(xy 295.91 109.22) (xy 312.42 109.22)
 		)
@@
 	(wire
 		(pts
+			(xy 154.94 492.76) (xy 177.8 492.76)
+		)
+		(stroke
+			(width 0)
+			(type default)
+		)
+	)
+	(wire
+		(pts
 			(xy 295.91 132.08) (xy 312.42 132.08)
 		)
@@
 		)
 	)
-	(hierarchical_label "RADIO_SD_DATA1"
+	(hierarchical_label "uP_SD2_DATA1"
 		(shape input)
 		(at 177.8 516.89 0)
@@
 		)
 	)
+	(hierarchical_label "uP_GPIO4_IO10"
+		(shape input)
+		(at 177.8 490.22 0)
+		(effects
+			(font
+				(size 1.27 1.27)
+			)
+			(justify left)
+		)
+	)
 	(hierarchical_label "uP_ENET1_RX_DATA0"
 		(shape input)
@@
 		)
 	)
-	(hierarchical_label "RADIO_SD_DATA2"
+	(hierarchical_label "uP_SD2_DATA2"
 		(shape input)
 		(at 177.8 519.43 0)
@@
 		)
 	)
+	(hierarchical_label "uP_GPIO4_IO11"
+		(shape input)
+		(at 177.8 500.38 0)
+		(effects
+			(font
+				(size 1.27 1.27)
+			)
+			(justify left)
+		)
+	)
 	(hierarchical_label "DRAM_SDQSO_N"
 		(shape input)
@@
 		)
 	)
-	(hierarchical_label "RADIO_SD_DATA3"
+	(hierarchical_label "uP_SD2_DATA3"
 		(shape input)
 		(at 177.8 521.97 0)
@@
 		)
 	)
-	(hierarchical_label "RADIO_SD_CLK"
+	(hierarchical_label "uP_SD2_CLK"
 		(shape input)
 		(at 177.8 495.3 0)
@@
 		)
 	)
+	(hierarchical_label "uP_GPIO4_IO12"
+		(shape input)
+		(at 177.8 502.92 0)
+		(effects
+			(font
+				(size 1.27 1.27)
+			)
+			(justify left)
+		)
+	)
 	(hierarchical_label "uP_SD1_DATA3"
 		(shape input)
@@
 		)
 	)
+	(hierarchical_label "uP_GPIO4_IO15"
+		(shape input)
+		(at 177.8 492.76 0)
+		(effects
+			(font
+				(size 1.27 1.27)
+			)
+			(justify left)
+		)
+	)
 	(hierarchical_label "DRAM_CS1_B"
 		(shape input)
@@
 		)
 	)
-	(hierarchical_label "RADIO_SD_CMD"
+	(hierarchical_label "uP_SD2_CMD"
 		(shape input)
 		(at 177.8 497.84 0)
@@
 		)
 	)
-	(hierarchical_label "RADIO_SD_DATA0"
+	(hierarchical_label "uP_SD2_DATA0"
 		(shape input)
 		(at 177.8 514.35 0)

Commit message: minor updates
Connections:
- net +1V8_RADIO is gone; now on net DCDC_3V3: U1.F4 (NVCC_CSI)
- net DCDC_3V3: now also U1.C4 (NVCC_SD1), U1.E7 (NVCC_NAND), U1.F13 (NVCC_ENET), U1.J13 (NVCC_GPIO)
- net GND: now also U1.A1 (VSS_1), U1.A17 (VSS_2), U1.C11 (VSS_5), U1.C15 (VSS_6), U1.C3 (VSS_3), U1.C7 (VSS_4), U1.E11 (VSS_8), U1.E8 (VSS_7), U1.F10 (VSS_13), U1.F11 (VSS_14), U1.F12 (VSS_15), U1.F6 (VSS_9), U1.F7 (VSS_10), U1.F8 (VSS_11), U1.F9 (VSS_12), U1.G12 (VSS_19), U1.G15 (VSS_20), U1.G3 (VSS_16), U1.G5 (VSS_17), U1.G7 (VSS_18), U1.H12 (VSS_22), U1.H7 (VSS_21), U1.J12 (VSS_25), U1.J5 (VSS_23), U1.J7 (VSS_24), U1.K12 (VSS_27), U1.K7 (VSS_26), U1.L12 (VSS_30), U1.L3 (VSS_28), U1.L7 (VSS_29), U1.M10 (VSS_34), U1.M11 (VSS_35), U1.M7 (VSS_31), U1.M8 (VSS_32), U1.M9 (VSS_33), U1.N3 (VSS_36), U1.N5 (VSS_37), U1.R11 (VSS_41), U1.R16 (VSS_42), U1.R17 (VSS_43), U1.R3 (VSS_38), U1.R5 (VSS_39), U1.R7 (VSS_40), U1.T14 (VSS_44), U1.U1 (VSS_45), U1.U14 (VSS_46), U1.U17 (VSS_47)

Commit message: Minor updates again!
Connections:
- net VDD_ARM_SOC: now reaches U1.H10 (VDD_SOC_IN_2)
- net VDD_ARM_SOC: now also U1.H9 (VDD_SOC_IN_1), U1.J10 (VDD_SOC_IN_4), U1.J9 (VDD_SOC_IN_3), U1.K10 (VDD_SOC_IN_6), U1.K9 (VDD_SOC_IN_5)
Changed lines of the file:
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@@
 	)
 	(junction
+		(at 68.58 60.96)
+		(diameter 0)
+		(color 0 0 0 0)
+	)
+	(junction
 		(at 195.58 328.93)
 		(diameter 0)
@@
 	)
 	(junction
+		(at 68.58 63.5)
+		(diameter 0)
+		(color 0 0 0 0)
+	)
+	(junction
 		(at 85.09 130.81)
 		(diameter 0)
@@
 	)
 	(junction
+		(at 68.58 66.04)
+		(diameter 0)
+		(color 0 0 0 0)
+	)
+	(junction
 		(at 200.66 148.59)
 		(diameter 0)
@@
 	)
 	(junction
+		(at 68.58 68.58)
+		(diameter 0)
+		(color 0 0 0 0)
+	)
+	(junction
 		(at 85.09 148.59)
 		(diameter 0)
@@
 	)
 	(junction
+		(at 68.58 58.42)
+		(diameter 0)
+		(color 0 0 0 0)
+	)
+	(junction
 		(at 200.66 151.13)
 		(diameter 0)
@@
 	(wire
 		(pts
+			(xy 68.58 60.96) (xy 68.58 63.5)
+		)
+		(stroke
+			(width 0)
+			(type default)
+		)
+	)
+	(wire
+		(pts
 			(xy 177.8 161.29) (xy 200.66 161.29)
 		)
@@
 	(wire
 		(pts
+			(xy 99.06 68.58) (xy 68.58 68.58)
+		)
+		(stroke
+			(width 0)
+			(type default)
+		)
+	)
+	(wire
+		(pts
 			(xy 179.07 261.62) (xy 217.17 261.62)
 		)
@@
 	(wire
 		(pts
+			(xy 68.58 66.04) (xy 68.58 68.58)
+		)
+		(stroke
+			(width 0)
+			(type default)
+		)
+	)
+	(wire
+		(pts
 			(xy 200.66 161.29) (xy 200.66 163.83)
 		)
@@
 	(wire
 		(pts
+			(xy 68.58 68.58) (xy 68.58 71.12)
+		)
+		(stroke
+			(width 0)
+			(type default)
+		)
+	)
+	(wire
+		(pts
 			(xy 774.7 176.53) (xy 774.7 189.23)
 		)
@@
 	(wire
 		(pts
+			(xy 99.06 60.96) (xy 68.58 60.96)
+		)
+		(stroke
+			(width 0)
+			(type default)
+		)
+	)
+	(wire
+		(pts
 			(xy 92.71 337.82) (xy 100.33 337.82)
 		)
@@
 	(wire
 		(pts
+			(xy 99.06 58.42) (xy 68.58 58.42)
+		)
+		(stroke
+			(width 0)
+			(type default)
+		)
+	)
+	(wire
+		(pts
 			(xy 179.07 265.43) (xy 217.17 265.43)
 		)
@@
 	(wire
 		(pts
+			(xy 99.06 66.04) (xy 68.58 66.04)
+		)
+		(stroke
+			(width 0)
+			(type default)
+		)
+	)
+	(wire
+		(pts
 			(xy 198.12 384.81) (xy 185.42 384.81)
 		)
@@
 	(wire
 		(pts
+			(xy 99.06 63.5) (xy 68.58 63.5)
+		)
+		(stroke
+			(width 0)
+			(type default)
+		)
+	)
+	(wire
+		(pts
 			(xy 449.58 445.77) (xy 467.36 445.77)
 		)
@@
 	(wire
 		(pts
+			(xy 68.58 63.5) (xy 68.58 66.04)
+		)
+		(stroke
+			(width 0)
+			(type default)
+		)
+	)
+	(wire
+		(pts
 			(xy 364.49 217.17) (xy 383.54 217.17)
 		)
@@
 	(wire
 		(pts
+			(xy 68.58 58.42) (xy 68.58 60.96)
+		)
+		(stroke
+			(width 0)
+			(type default)
+		)
+	)
+	(wire
+		(pts
 			(xy 92.71 337.82) (xy 92.71 346.71)
 		)
@@
 	(wire
 		(pts
+			(xy 99.06 71.12) (xy 68.58 71.12)
+		)
+		(stroke
+			(width 0)
+			(type default)
+		)
+	)
+	(wire
+		(pts
 			(xy 71.12 254) (xy 100.33 254)
 		)
@@
 	(wire
 		(pts
+			(xy 68.58 50.8) (xy 68.58 58.42)
+		)
+		(stroke
+			(width 0)
+			(type default)
+		)
+	)
+	(wire
+		(pts
 			(xy 200.66 168.91) (xy 200.66 171.45)
 		)
@@
 					(unit 1)
 				)
+			)
+		)
+	)
+	(symbol
+		(lib_id "power:+1V35")
+		(at 68.58 50.8 0)
+		(unit 1)
+		(exclude_from_sim no)
+		(in_bom yes)
+		(on_board yes)
+		(dnp no)
+		(fields_autoplaced yes)
+		(property "Reference" "#PWR0146"
+			(at 68.58 54.61 0)
+			(effects
+				(font
+					(size 1.27 1.27)
+				)
+				(hide yes)
+			)
+		)
+		(property "Value" "VDD_ARM_SOC"
+			(at 68.58 45.72 0)
+			(effects
+				(font
+					(size 1.27 1.27)
+				)
+			)
+		)
+		(property "Footprint" ""
+			(at 68.58 50.8 0)
+			(effects
+				(font
+					(size 1.27 1.27)
+				)
+				(hide yes)
+			)
+		)
+		(property "Datasheet" ""
+			(at 68.58 50.8 0)
+			(effects
+				(font
+					(size 1.27 1.27)
+				)
+				(hide yes)
+			)
+		)
+		(property "Description" "Power symbol creates a global label with name \"+1V35\""
+			(at 68.58 50.8 0)
+			(effects
+				(font
+					(size 1.27 1.27)
+				)
+				(hide yes)
+			)
+		)
+		(pin "1"
+		)
+		(instances
+			(project "NXP_SBC"
+				(path "/e82fc437-413b-4185-b609-66f66e24e498/0ea4c833-27a6-4c6c-939d-80a3ef0aae04"
+					(reference "#PWR0146")
+					(unit 1)
+				)
