File: NXP/Hardware/NXP_SOM/NXP_SOM/Memory_sch.kicad_sch (KiCad schematic)
At the start: 38 parts, among them J1 Micro_SD_Card_Det2, U2 MT41K256M16TW-107_P_TR

Commit message: connected RAM to SOM
Parts:
- removed D1, D2, D3, D4, D5, D6, D7: PESD3V3Z1BSFYL, symbol Chase_Diode:PESD3V3Z1BSFYL
- removed J1: Micro_SD_Card_Det2, Connector_Card:microSD_HC_Molex_104031-0811, symbol Connector:Micro_SD_Card_Det2
- removed R1, R2, R3, R4, R5, R6: 47k, Resistor_SMD:R_01005_0402Metric, symbol Device:R_Small
Connections:
- net RAM_DQ9: no longer C42.1, C43.1
- net RAM_UDQS: now also C42.1, C43.1
Other:
- note removed: "SD CARD HOLDER"
