File: NXP/Hardware/NXP_SOM/NXP_SOM/NXP_SOM.kicad_sch (KiCad schematic)
At the start: 0 parts

Commit message: connected RAM to SOM
Connections:
- no-connect marks 0 -> 4
Other:
- added sheet Ethernet_PHY (Ethernet.kicad_sch)
- sheet Processor ports: added DRAM_ADDR00, DRAM_ADDR01, DRAM_ADDR02, DRAM_ADDR03, DRAM_ADDR04, DRAM_ADDR05, DRAM_ADDR06, DRAM_ADDR07, DRAM_ADDR08, DRAM_ADDR09, DRAM_ADDR10, DRAM_ADDR11, DRAM_ADDR12, DRAM_ADDR13, DRAM_ADDR14, DRAM_ADDR15, DRAM_CAS_B, DRAM_CS0_B, DRAM_CS1_B, DRAM_DATA0, DRAM_DATA1, DRAM_DATA10, DRAM_DATA11, DRAM_DATA12, DRAM_DATA13, DRAM_DATA14, DRAM_DATA15, DRAM_DATA2, DRAM_DATA3, DRAM_DATA4, DRAM_DATA5, DRAM_DATA6, DRAM_DATA7, DRAM_DATA8, DRAM_DATA9, DRAM_DQM0, DRAM_DQM1, DRAM_ODT0, DRAM_ODT1, DRAM_RAS_B, DRAM_RESET, DRAM_SDBA0, DRAM_SDBA1, DRAM_SDBA2, DRAM_SDCLK0_N, DRAM_SDCLK0_P, DRAM_SDKE0, DRAM_SDKE1, DRAM_SDQS0_P, DRAM_SDQS1_N, DRAM_SDQS1_P, DRAM_SDQSO_N, DRAM_SDWE_B, DRAM_VREF; removed none
- sheet RAM ports: added DDR_VREF, RAM_ADDR0, RAM_ADDR1, RAM_ADDR10, RAM_ADDR11, RAM_ADDR12, RAM_ADDR13, RAM_ADDR14, RAM_ADDR2, RAM_ADDR3, RAM_ADDR4, RAM_ADDR5, RAM_ADDR6, RAM_ADDR7, RAM_ADDR8, RAM_ADDR9, RAM_BANK_ADDR0, RAM_BANK_ADDR1, RAM_BANK_ADDR2, RAM_CAS#, RAM_CK, RAM_CK#, RAM_CKE, RAM_CS#, RAM_DQ0, RAM_DQ1, RAM_DQ10, RAM_DQ11, RAM_DQ12, RAM_DQ13, RAM_DQ14, RAM_DQ15, RAM_DQ2, RAM_DQ3, RAM_DQ4, RAM_DQ5, RAM_DQ6, RAM_DQ7, RAM_DQ8, RAM_DQ9, RAM_LDM, RAM_LDQS, RAM_LDQS#, RAM_ODT, RAM_RAS#, RAM_RESET, RAM_UDM, RAM_UDQS, RAM_UDQS#, RAM_WE#; removed none
