File: NXP/Hardware/NXP_SOM/NXP_SOM/Processor.kicad_sch (KiCad schematic)
At the start: 51 parts, among them U1 MCIMX6Y2DVM09AB

Commit message: connected RAM to SOM
Parts:
- added C1, C2, C68, C69, C70: 220nF, Capacitor_SMD:C_0603_1608Metric_Pad1.08x0.95mm_HandSolder, symbol Device:C_Small
Connections:
- net +1V8_RADIO: now also C108.1
- net DCDC_3V3: now also U1.C4 (NVCC_SD1), U1.E7 (NVCC_NAND), U1.F13 (NVCC_ENET), U1.J13 (NVCC_GPIO), U1.L13 (VDDA_ADC_3P3), C1.1, C2.1, C68.1, C69.1, C70.1
- net GND: now also C108.2, C1.2, C2.2, C68.2, C69.2, C70.2
Other:
- moved on the sheet: C55, U1F, U1H, U1I, U1J
